Commit message: Rover model updated (replaced by polaris)

File: ardupilot_sitl_gazebo_plugin/urdf/rover.urdf (robot description, URDF)
Before this commit: robot rover, 11 links, 10 joints
Links:
- removed link rover__back_left_wheel
- removed link rover__back_right_wheel
- removed link rover__bottom_cam_link
- removed link rover__brake_pedal
- removed link rover__chassis
- removed link rover__front_cam_link
- removed link rover__front_left_wheel
- removed link rover__front_right_wheel
- removed link rover__gas_pedal
- removed link rover__imu_link
- removed link rover__steering_wheel
- added link chassis, mass 720.0; collision box size=1.34 1.65746 0.06; visual box size=1.34 1.65746 0.06
- added link front_left_wheel, mass 12; collision cylinder length=0.2794 radius=0.3175; visual cylinder length=0.2794 radius=0.3175
- added link front_left_wheel_steering_block, mass 1; collision cylinder length=0.01 radius=0.05
- added link front_right_wheel, mass 12; collision cylinder length=0.2794 radius=0.3175; visual cylinder length=0.2794 radius=0.3175
- added link front_right_wheel_steering_block, mass 1; collision cylinder length=0.01 radius=0.05
- added link rear_left_wheel, mass 12; collision cylinder length=0.2794 radius=0.3175; visual cylinder length=0.2794 radius=0.3175
- added link rear_right_wheel, mass 12; collision cylinder length=0.2794 radius=0.3175; visual cylinder length=0.2794 radius=0.3175
Joints:
- removed joint rover__back_left_joint
- removed joint rover__back_right_joint
- removed joint rover__bottom_cam_joint
- removed joint rover__brake_joint
- removed joint rover__front_cam_joint
- removed joint rover__front_left_joint
- removed joint rover__front_right_joint
- removed joint rover__gas_joint
- removed joint rover__imu_joint
- removed joint rover__steering_joint
- added joint front_left_steering_joint: type revolute, parent chassis, child front_left_wheel_steering_block, origin xyz=1.20222  0.5      0.35515 rpy=1.57079  0       0, axis 0  1  0, limit lower=-0.7727 upper=0.7727 effort=10.0 velocity=0.0
- added joint front_left_wheel_joint: type revolute, parent front_left_wheel_steering_block, child front_left_wheel, origin xyz=0      -0.00818 -0.21562 rpy=-3.09079  0       0, axis 0.00000000e+00   8.30000000e-04   1.00000000e+00, limit lower=0 upper=0 effort=10.0 velocity=0
- added joint front_right_steering_joint: type revolute, parent chassis, child front_right_wheel_steering_block, origin xyz=1.20222 -0.5      0.35515 rpy=1.57079  0       0, axis 0  1  0, limit lower=-0.7727 upper=0.7727 effort=10.0 velocity=0.0
- added joint front_right_wheel_joint: type revolute, parent front_right_wheel_steering_block, child front_right_wheel, origin xyz=0      -0.00818  0.21562 rpy=-0.05079  0       0, axis 0.00000000e+00   8.30000000e-04  -1.00000000e+00, limit lower=0 upper=0 effort=0 velocity=0
- added joint rear_left_wheel_joint: type revolute, parent chassis, child rear_left_wheel, origin xyz=-0.99377  0.71562  0.34697 rpy=-1.52  0    0, axis 0.00000000e+00   8.30000000e-04   1.00000000e+00, limit lower=0 upper=0 effort=0 velocity=0
- added joint rear_right_wheel_joint: type revolute, parent chassis, child rear_right_wheel, origin xyz=-0.99377 -0.61574  0.34189 rpy=1.52  0    0, axis 0.00000000e+00   8.30000000e-04  -1.00000000e+00, limit lower=0 upper=0 effort=0 velocity=0

Commit message: Normalize yaw and throttle values

File: ardupilot_sitl_gazebo_plugin/urdf/rover.urdf (robot description, URDF)
Before this commit: robot rover, 7 links, 6 joints
Links:
- link chassis: mass 720.0 -> 500.0; geometry collision box size=1.34 1.0 0.06; visual box size=1.34 1.0 0.06

Commit message: Add link for the IMU

File: ardupilot_sitl_gazebo_plugin/urdf/rover.urdf (robot description, URDF)
Before this commit: robot rover, 7 links, 6 joints
Links:
- added link imu, mass 0.00001; collision box size=0.02 0.02 0.02; visual box size=0.02 0.02 0.02
Joints:
- added joint imu_joint: type fixed, parent chassis, child imu

Commit message: Fix style

File: ardupilot_sitl_gazebo_plugin/urdf/rover.urdf (robot description, URDF)
Before this commit: robot rover, 8 links, 7 joints
Joints:
- joint front_left_steering_joint: origin xyz=1.20222  0.5      0.35515 rpy=1.57079  0       0 -> xyz=1.20222  0.5 0.35515 rpy=1.57079 0 0
- joint front_left_wheel_joint: axis 0.00000000e+00   8.30000000e-04   1.00000000e+00 -> 0.00000000e+00 8.30000000e-04 1.00000000e+00; origin xyz=0      -0.00818 -0.21562 rpy=-3.09079  0       0 -> xyz=0 -0.00818 -0.21562 rpy=-3.09079 0 0
- joint front_right_steering_joint: origin xyz=1.20222 -0.5      0.35515 rpy=1.57079  0       0 -> xyz=1.20222 -0.5 0.35515 rpy=1.57079 0 0
- joint front_right_wheel_joint: axis 0.00000000e+00   8.30000000e-04  -1.00000000e+00 -> 0.00000000e+00 8.30000000e-04 -1.00000000e+00; origin xyz=0      -0.00818  0.21562 rpy=-0.05079  0       0 -> xyz=0 -0.00818 0.21562 rpy=-0.05079 0 0
- joint rear_left_wheel_joint: axis 0.00000000e+00   8.30000000e-04   1.00000000e+00 -> 0.00000000e+00 8.30000000e-04 1.00000000e+00; origin xyz=-0.99377  0.71562  0.34697 rpy=-1.52  0    0 -> xyz=-0.99377 0.71562 0.34697 rpy=-1.52 0 0
- joint rear_right_wheel_joint: axis 0.00000000e+00   8.30000000e-04  -1.00000000e+00 -> 0.00000000e+00 8.30000000e-04 -1.00000000e+00; origin xyz=-0.99377 -0.61574  0.34189 rpy=1.52  0    0 -> xyz=-0.99377 -0.61574 0.34189 rpy=1.52 0 0

Commit message: Apply meshes to the rover

File: ardupilot_sitl_gazebo_plugin/urdf/rover.urdf (robot description, URDF)
Before this commit: robot rover, 8 links, 7 joints
Links:
- link chassis: geometry collision box size=1.34 1.0 0.06; visual mesh filename=package://ardupilot_sitl_gazebo_plugin/meshes/meshes_rover/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 scale=0.0055 0.0055 0.0055
- link front_left_wheel: geometry collision cylinder length=0.2794 radius=0.3175; visual mesh filename=package://ardupilot_sitl_gazebo_plugin/meshes/meshes_rover/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 scale=0.007 0.007 0.007
- link front_right_wheel: geometry collision cylinder length=0.2794 radius=0.3175; visual mesh filename=package://ardupilot_sitl_gazebo_plugin/meshes/meshes_rover/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 scale=0.007 0.007 0.007
- link rear_left_wheel: geometry collision cylinder length=0.2794 radius=0.3175; visual mesh filename=package://ardupilot_sitl_gazebo_plugin/meshes/meshes_rover/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 scale=0.007 0.007 0.007
- link rear_right_wheel: geometry collision cylinder length=0.2794 radius=0.3175; visual mesh filename=package://ardupilot_sitl_gazebo_plugin/meshes/meshes_rover/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 scale=0.007 0.007 0.007
Joints:
- joint rear_left_wheel_joint: origin xyz=-0.99377 0.71562 0.34697 rpy=-1.52 0 0 -> xyz=-0.75 0.75 0.34697 rpy=-1.52 0 0
- joint rear_right_wheel_joint: origin xyz=-0.99377 -0.61574 0.34189 rpy=1.52 0 0 -> xyz=-0.75 -0.75 0.34189 rpy=1.52 0 0

Commit message: Add parameters. Fix #7 and fix #5

File: ardupilot_sitl_gazebo_plugin/urdf/rover.urdf (robot description, URDF)
Before this commit: robot rover, 8 links, 7 joints
Joints:
- joint front_left_wheel_joint: origin xyz=0 -0.00818 -0.21562 rpy=-3.09079 0 0 -> xyz=0 -0.00818 -0.21562 rpy=0 0 0
- joint front_right_wheel_joint: origin xyz=0 -0.00818 0.21562 rpy=-0.05079 0 0 -> xyz=0 -0.00818 0.21562 rpy=0 0 0
- joint rear_left_wheel_joint: origin xyz=-0.75 0.75 0.34697 rpy=-1.52 0 0 -> xyz=-0.75 0.75 0.34697 rpy=-1.57079 0 0
- joint rear_right_wheel_joint: origin xyz=-0.75 -0.75 0.34189 rpy=1.52 0 0 -> xyz=-0.75 -0.75 0.34189 rpy=1.55079 0 0

Commit message: Fix GPS jumps and front left wheel orientation - Fixed GPS jumps by increasing update rate - Fixed front left wheel orientation permanently

File: ardupilot_sitl_gazebo_plugin/urdf/rover.urdf (robot description, URDF)
Before this commit: robot rover, 8 links, 7 joints
Links:
- removed link imu
Joints:
- removed joint imu_joint
- joint front_left_steering_joint: axis 0  1  0 -> 0  -1  0; origin xyz=1.20222  0.5 0.35515 rpy=1.57079 0 0 -> xyz=1.20222  0.5 0.35515 rpy=-1.52 0 0
- joint front_left_wheel_joint: origin xyz=0 -0.00818 -0.21562 rpy=0 0 0 -> xyz=0 -0.00818 0.21562 rpy=0 0 0
- joint front_right_steering_joint: origin xyz=1.20222 -0.5 0.35515 rpy=1.57079 0 0 -> xyz=1.20222 -0.5 0.35515 rpy=1.52 0 0
- joint rear_left_wheel_joint: origin xyz=-0.75 0.75 0.34697 rpy=-1.57079 0 0 -> xyz=-0.75 0.75 0.34697 rpy=-1.52 0 0
- joint rear_right_wheel_joint: origin xyz=-0.75 -0.75 0.34189 rpy=1.55079 0 0 -> xyz=-0.75 -0.75 0.34189 rpy=1.52 0 0

Commit message: Fix slightly the displacement of the vehicle

File: ardupilot_sitl_gazebo_plugin/urdf/rover.urdf (robot description, URDF)
Before this commit: robot rover, 7 links, 6 joints
Joints:
- joint rear_right_wheel_joint: origin xyz=-0.75 -0.75 0.34189 rpy=1.52 0 0 -> xyz=-0.75 -0.75 0.34697 rpy=1.52 0 0

Commit message: Change Yaw direction

File: ardupilot_sitl_gazebo_plugin/urdf/rover.urdf (robot description, URDF)
Before this commit: robot rover, 7 links, 6 joints
Links:
- added link base_link
Joints:
- added joint base_joint: type fixed, parent base_link, child chassis, origin xyz=0 0 0 rpy=0 0 0
- joint front_left_steering_joint: limit lower=-0.7727 upper=0.7727 effort=10.0 velocity=0.0 -> lower=-0.7727 upper=0.7727 effort=0 velocity=0.0
- joint front_left_wheel_joint: limit lower=0 upper=0 effort=10.0 velocity=0 -> lower=0 upper=0 effort=0 velocity=0
- joint front_right_steering_joint: limit lower=-0.7727 upper=0.7727 effort=10.0 velocity=0.0 -> lower=-0.7727 upper=0.7727 effort=0 velocity=0.0

Commit message: Trying to fix #10

File: ardupilot_sitl_gazebo_plugin/urdf/rover.urdf (robot description, URDF)
Before this commit: robot rover, 8 links, 7 joints
Links:
- removed link base_link
- added link imu, mass 0.00001; collision box size=0.02 0.02 0.02; visual box size=0.02 0.02 0.02
Joints:
- removed joint base_joint
- added joint imu_joint: type fixed, parent chassis, child imu

Commit message: Trying to fix #10

File: ardupilot_sitl_gazebo_plugin/urdf/rover.urdf (robot description, URDF)
Before this commit: robot rover, 8 links, 7 joints
Links:
- link chassis: geometry collision box size=1.34 1.0 0.06
- link front_left_wheel: geometry collision cylinder length=0.2794 radius=0.3175
- link front_right_wheel: geometry collision cylinder length=0.2794 radius=0.3175
- link rear_left_wheel: geometry collision cylinder length=0.2794 radius=0.3175
- link rear_right_wheel: geometry collision cylinder length=0.2794 radius=0.3175

Commit message: Still testing

File: ardupilot_sitl_gazebo_plugin/urdf/rover.urdf (robot description, URDF)
Before this commit: robot rover, 8 links, 7 joints
Joints:
- joint front_left_steering_joint: axis 0  -1  0 -> 0  1  0; origin xyz=1.20222  0.5 0.35515 rpy=-1.52 0 0 -> xyz=1.20222  0.5 0.35515 rpy=1.52 0 0
- joint front_left_wheel_joint: origin xyz=0 -0.00818 0.21562 rpy=0 0 0 -> xyz=0 -0.00818 -0.21562 rpy=0 0 0

Commit message: Temporally fix #10 Remove visuals from rear wheels so that GUIDED mode and GPS work.

File: ardupilot_sitl_gazebo_plugin/urdf/rover.urdf (robot description, URDF)
Before this commit: robot rover, 7 links, 6 joints
Links:
- link rear_left_wheel: geometry collision cylinder length=0.2794 radius=0.3175; visual cylinder length=0.2794 radius=0.3175
- link rear_right_wheel: geometry collision cylinder length=0.2794 radius=0.3175; visual cylinder length=0.2794 radius=0.3175

Commit message: Remove visuals and adjust camera and laser - Remove visuals to avoid issues with the GPS - Adjust camera position and resolution - Adjust laser position and fov

File: ardupilot_sitl_gazebo_plugin/urdf/rover.urdf (robot description, URDF)
Before this commit: robot rover, 7 links, 6 joints
Links:
- link chassis: geometry collision box size=1.34 1.0 0.06; visual box size=1.34 1.0 0.06
- link front_left_wheel: geometry collision cylinder length=0.2794 radius=0.3175; visual cylinder length=0.2794 radius=0.3175
- link front_right_wheel: geometry collision cylinder length=0.2794 radius=0.3175; visual cylinder length=0.2794 radius=0.3175

Commit message: Fix wheels block

File: ardupilot_sitl_gazebo_plugin/urdf/rover.urdf (robot description, URDF)
Before this commit: robot rover, 7 links, 6 joints
Links:
- link front_left_wheel: geometry collision cylinder length=0.2794 radius=0.3175; visual mesh filename=package://ardupilot_sitl_gazebo_plugin/meshes/meshes_rover/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 scale=0.007 0.007 0.007
- link front_right_wheel: geometry collision cylinder length=0.2794 radius=0.3175; visual mesh filename=package://ardupilot_sitl_gazebo_plugin/meshes/meshes_rover/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 scale=0.007 0.007 0.007
- link rear_left_wheel: geometry collision cylinder length=0.2794 radius=0.3175; visual mesh filename=package://ardupilot_sitl_gazebo_plugin/meshes/meshes_rover/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 scale=0.007 0.007 0.007
- link rear_right_wheel: geometry collision cylinder length=0.2794 radius=0.3175; visual mesh filename=package://ardupilot_sitl_gazebo_plugin/meshes/meshes_rover/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 scale=0.007 0.007 0.007
Joints:
- joint front_left_wheel_joint: origin xyz=0 -0.00818 0.21562 rpy=0 0 0 -> xyz=0 0 0.21562 rpy=0 0 0
- joint front_right_wheel_joint: origin xyz=0 -0.00818 0.21562 rpy=0 0 0 -> xyz=0 0 0.21562 rpy=0 0 0
